Commit message: 「xarco」ではなく「xacro」です

File: world_setup/urdf/robot.urdf (robot description, URDF)
Before this commit: robot my_robot, 3 links, 2 joints
Links:
- link camera_link: geometry collision box size=${camera_size}; visual box size=${camera_size}
- link link_arm: geometry collision box size=${link_arm_size}; visual box size=${link_arm_size}
- link link_chassis: geometry collision box size=${link_chassis_size}; visual box size=${link_chassis_size}
Joints:
- joint camera_joint: origin xyz=1 0 1 rpy=0 0 0 -> xyz=0.2 0 0.5 rpy=0 0 0
- joint joint_1: origin xyz=0.6 0 0.8 rpy=0 0 0 -> xyz=0.6 0 0.5 rpy=0 0 0

Commit message: wheels & models

File: world_setup/urdf/robot.urdf (robot description, URDF)
Before this commit: robot my_robot, 3 links, 2 joints
Links:
- added link link_left_wheel, mass 0.2; collision cylinder length=${wheel_length} radius=${wheel_radius}; visual cylinder length=${wheel_length} radius=${wheel_radius}
- added link link_left_wheel_f, mass 0.2; collision cylinder length=${wheel_length} radius=${wheel_radius}; visual cylinder length=${wheel_length} radius=${wheel_radius}
- added link link_right_wheel, mass 0.2; collision cylinder length=${wheel_length} radius=${wheel_radius}; visual cylinder length=${wheel_length} radius=${wheel_radius}
- added link link_right_wheel_f, mass 0.2; collision cylinder length=${wheel_length} radius=${wheel_radius}; visual cylinder length=${wheel_length} radius=${wheel_radius}
Joints:
- added joint joint_left_wheel: type continuous, parent link_chassis, child link_left_wheel, origin xyz=-0.8 -0.5 0 rpy=0 0 0, axis 0 1 0, limit effort=10000 velocity=1000
- added joint joint_left_wheel_f: type continuous, parent link_chassis, child link_left_wheel_f, origin xyz=0.8 -0.5 0 rpy=0 0 0, axis 0 1 0, limit effort=10000 velocity=1000
- added joint joint_right_wheel: type continuous, parent link_chassis, child link_right_wheel, origin xyz=-0.8 0.5 0 rpy=0 0 0, axis 0 1 0, limit effort=10000 velocity=1000
- added joint joint_right_wheel_f: type continuous, parent link_chassis, child link_right_wheel_f, origin xyz=0.8 0.5 0 rpy=0 0 0, axis 0 1 0, limit effort=10000 velocity=1000
- joint joint_1: type continuous -> fixed
