Commit message: add rover2 & movers

File: test_world/urdf/macros.xacro (robot description, xacro)
@@ -8,5 +8,5 @@
               <inertia ixx="0.000526666666667" ixy="0" ixz="0" iyy="0.000526666666667" iyz="0" izz="0.001"/>
             </inertial>
-            <collision name="link_right_wheel_collision">
+            <collision name="${name}_collision">
               <origin rpy="0 1.5707 1.5707" xyz="0 0 0"/>
               <geometry>
@@ -22,8 +22,8 @@
         </link>
     </xacro:macro>
-    <xacro:macro name="joint_wheel" params="name child origin_xyz">
+    <xacro:macro name="joint_wheel" params="name child origin_xyz parent">
       <joint name="${name}" type="continuous">
         <origin rpy="0 0 0" xyz="${origin_xyz}"/>
-        <parent link="link_chassis"/>
+        <parent link="${parent}"/>
         <child link="${child}"/>
         <axis rpy="0 0 0" xyz="0 1 0"/>

File: test_world/urdf/robot2/robot.urdf (robot description, URDF)
Before this commit: robot m2wr, 2 links, 1 joints
Links:
- removed link link_chassis
- added link caster, mass 0.2; collision cylinder length=0.1 radius=0.05; visual cylinder length=0.1 radius=0.05
- added link link_chassis2, mass 5; collision box size=0.5 0.3 0.07; visual box size=0.5 0.3 0.07
Joints:
- added joint joint_caster: type continuous, parent link_chassis2, child caster, origin xyz=0.35 0 -0.05 rpy=0 0 0, axis 0 1 0, limit effort=10000 velocity=1000
- joint joint_sensor_laser: parent link_chassis -> link_chassis2

Commit message: improve surface

File: test_world/urdf/macros.xacro (robot description, xacro)
@@ -5,17 +5,17 @@
             <inertial>
               <mass value="0.2"/>
-              <origin rpy="0 1.5707 1.5707" xyz="0 0 0"/>
-              <inertia ixx="0.000526666666667" ixy="0" ixz="0" iyy="0.000526666666667" iyz="0" izz="0.001"/>
+              <origin rpy="0 1.570796 1.570796" xyz="0 0 0"/>
+              <xacro:cylinder_inertia mass="0.2" l="0.03" r="0.1" />
             </inertial>
             <collision name="${name}_collision">
-              <origin rpy="0 1.5707 1.5707" xyz="0 0 0"/>
+              <origin rpy="0 1.570796 1.570796" xyz="0 0 0"/>
               <geometry>
-                <cylinder length="0.04" radius="0.1"/>
+                <cylinder length="0.03" radius="0.1"/>
               </geometry>
             </collision>
             <visual name="${name}_visual">
-              <origin rpy="0 1.5707 1.5707" xyz="0 0 0"/>
+              <origin rpy="0 1.570796 1.570796" xyz="0 0 0"/>
               <geometry>
-                <cylinder length="0.04" radius="0.1"/>
+                <cylinder length="0.03" radius="0.1"/>
               </geometry>
             </visual>

File: test_world/urdf/robot1/robot.urdf (robot description, URDF)
Before this commit: robot m2wr, 3 links, 2 joints
Links:
- removed link caster
- link link_chassis: geometry collision box size=0.5 0.3 0.07; collision sphere radius=0.05
Joints:
- removed joint joint_caster
