Commit message: service2 add path

File: test_world/urdf/robot2/robot.urdf (robot description, URDF)
Before this commit: robot m2wr2, 3 links, 2 joints
Links:
- removed link caster
- added link caster1, mass 0.2; collision cylinder length=0.02 radius=0.05; visual cylinder length=0.02 radius=0.05
- added link caster2, mass 0.2; collision cylinder length=0.03 radius=0.04; visual cylinder length=0.03 radius=0.04
Joints:
- removed joint joint_caster
- added joint joint_caster1: type continuous, parent link_chassis2, child caster1, origin xyz=0.25 0 -0.05 rpy=0 0 0, axis 0 0 1, limit effort=10000 velocity=1000
- added joint joint_caster2: type continuous, parent caster1, child caster2, origin xyz=0 0 0 rpy=0 0 0, axis 0 1 0, limit effort=10000 velocity=1000

Commit message: add interval correction

File: test_world/urdf/robot2/robot.urdf (robot description, URDF)
Before this commit: robot m2wr2, 4 links, 3 joints
Links:
- removed link caster1
- removed link caster2
- link link_chassis2: geometry collision box size=0.5 0.3 0.07; collision sphere radius=0.05
Joints:
- removed joint joint_caster1
- removed joint joint_caster2
